File: hardware/debugino.sch (EAGLE design)
At the start: 36 parts, among them Q1 12MHz, U2 ATMEGA328P-AU, U3 STM32F103CBT6, X1 MINI-USB-SCHIELD-32005-301

Commit message: Hardware for current measurement
Parts:
- added R12: 0.47R, custom:RESISTOR0805
- added R13: 1K5, custom:RESISTOR0603
- added U1: ZXCT1107SA-7, Diodes_Inc_By_element14_Batch_1:ZXCT1107SA-7
- R3, R4: value 1K -> 1K5
- R5, R6, R7, R8, R9: value 1k -> 1K5
Connections:
- new net +5V: C5.2, C6.2, J1.13, J2.2, R10.2, R12.2, U1.S-, U2.AVCC, U2.VCC, U2.VCC_2
- new net CURRENT: R13.1, U1.OUT, U3.PA3
- net GND: now also R13.2
- net VCC: now also R12.1, U1.S+; no longer C5.2, C6.2, J1.13, J2.2, R10.2, U2.AVCC, U2.VCC, U2.VCC_2
Other:
- note added: "Current measurement"
- moved on the sheet: F1, JP1, R1, R2, X1G$1
